Commit message: changed the urdf shape and join wk 7

File: genetic-algo-wk7/103.urdf (robot description, URDF)
Before this commit: robot myfirst, 2 links, 1 joints
Links:
- link sub_link: geometry collision cylinder length=0.6 radius=0.25; visual cylinder length=1 radius=0.1
Joints:
- joint base_to_sub: origin xyz=0 0 2.5 rpy=0 0 0 -> xyz=0 0.5 0 rpy=0 0 0; type revolute -> fixed
