Commit message: completed wk 8 activities changed the start.py

File: genetic-algo-wk8/wk3_end/test.urdf (robot description, URDF)
Before this commit: robot pepe, 15 links, 14 joints
Links:
- removed link 18
- removed link 29
- removed link 314
- removed link 37
- removed link 410
- removed link 411
- removed link 412
- removed link 413
- removed link 43
- removed link 44
- removed link 45
- removed link 46
- link 0: mass 1.2714566256624342 -> 1.1799171829958945; geometry collision cylinder length=0.6564084478039316 radius=0.7564212931887703; visual cylinder length=0.6564084478039316 radius=0.7564212931887703
- link 11: mass 0.4686701816333142 -> 0.05575835605967076; geometry collision cylinder length=0.22458029278200597 radius=0.28112160407444176; visual cylinder length=0.22458029278200597 radius=0.28112160407444176
- link 22: mass 0.7127293767372701 -> 0.09776460197075584; geometry collision cylinder length=0.6888501617099307 radius=0.21254627570448137; visual cylinder length=0.6888501617099307 radius=0.21254627570448137
Joints:
- removed joint 18_to_0
- removed joint 22_to_11
- removed joint 29_to_18
- removed joint 314_to_18
- removed joint 37_to_11
- removed joint 410_to_29
- removed joint 411_to_29
- removed joint 412_to_29
- removed joint 413_to_29
- removed joint 43_to_22
- removed joint 44_to_22
- removed joint 45_to_22
- removed joint 46_to_22
- added joint 22_to_0: type revolute, parent 0, child 22, origin xyz=0.23070946088005573 0.3372727583056099 0.9325378972382061 rpy=14.214528899812851 2.9921759752238684 1.2725719396311717, axis 1 0 0, limit lower=3.1415 upper=-3.1415 effort=1 velocity=1
- joint 11_to_0: origin xyz=0.5681223835788212 0.577980929657178 0.6057434120973962 rpy=5.727449388796838 5.818573912158904 1.7343350493282466 -> xyz=0.48815185230067804 0.5577554014220211 0.3592930529047639 rpy=10.410252862655849 2.3906155151984363 1.1446274652724877
