Commit message: updated the cw-envt and prepare_shapes to have my new code.

File: midterm-src-practice1/test.urdf (robot description, URDF)
Before this commit: robot pepe, 5 links, 4 joints
Links:
- removed link 12
- added link 22, mass 1.1389781359050966; collision cylinder length=1.5620240224464608 radius=0.48176905728716923; visual cylinder length=1.5620240224464608 radius=0.48176905728716923
- link 0: mass 0.08882193011447076 -> 1.722182365839306; geometry collision cylinder length=0.8619765257516752 radius=0.7974746987959628; visual cylinder length=0.8619765257516752 radius=0.7974746987959628
- link 11: mass 1.3629571017358157 -> 0.3657396403654328; geometry collision cylinder length=0.39591965389582406 radius=0.542259975153046; visual cylinder length=0.39591965389582406 radius=0.542259975153046
- link 13: mass 1.3629571017358157 -> 0.3657396403654328; geometry collision cylinder length=0.39591965389582406 radius=0.542259975153046; visual cylinder length=0.39591965389582406 radius=0.542259975153046
- link 24: mass 0.00927975494390793 -> 1.1389781359050966; geometry collision cylinder length=1.5620240224464608 radius=0.48176905728716923; visual cylinder length=1.5620240224464608 radius=0.48176905728716923
Joints:
- removed joint 12_to_0
- removed joint 24_to_0
- added joint 22_to_11: type revolute, parent 11, child 22, origin xyz=0.5086791799572757 0.6428086020897853 0.8283257935337676 rpy=11.32233760503962 0.9311136338179692 5.752138905189514, axis 0 0 1, limit lower=3.1415 upper=-3.1415 effort=1 velocity=1
- added joint 24_to_13: type revolute, parent 13, child 24, origin xyz=0.5086791799572757 0.6428086020897853 0.8283257935337676 rpy=11.32233760503962 0.9311136338179692 5.752138905189514, axis 0 0 1, limit lower=3.1415 upper=-3.1415 effort=1 velocity=1
- joint 11_to_0: axis 0 0 1 -> 0 1 0; origin xyz=0.13758607675745194 0.9350807390271525 0.7734982986138889 rpy=1.1448832225386056 4.335027266637536 1.6623373384868418 -> xyz=0.29904373405881135 0.01924679754309011 0.8123623879416968 rpy=11.546230044354902 0.14043467431111878 0.7744587835114084
- joint 13_to_0: axis 0 0 1 -> 0 1 0; origin xyz=0.13758607675745194 0.9350807390271525 0.7734982986138889 rpy=2.2897664450772113 4.335027266637536 1.6623373384868418 -> xyz=0.29904373405881135 0.01924679754309011 0.8123623879416968 rpy=17.319345066532353 0.14043467431111878 0.7744587835114084
