Commit message: combined the old realtime with the new make-arena code - changed the test_ga_no_threads.py to create some genomes and changed the iteration to 5

File: midterm-src-practice1/temp0.urdf (robot description, URDF)
Before this commit: robot pepe, 7 links, 6 joints
Links:
- link 11: mass 0.05557281936211409 -> 0.26446729291381127; geometry collision cylinder length=0.2532065960551713 radius=0.5765985436187973; visual cylinder length=0.2532065960551713 radius=0.5765985436187973
- link 14: mass 0.05557281936211409 -> 0.26446729291381127; geometry collision cylinder length=0.2532065960551713 radius=0.5765985436187973; visual cylinder length=0.2532065960551713 radius=0.5765985436187973
Joints:
- joint 11_to_0: origin xyz=0.9519997554499254 0.8346274683241105 0.9807371605957307 rpy=2.346661014776726 1.781064725250609 1.5965217213472793 -> xyz=0.9999 0.8346274683241105 0.9807371605957307 rpy=2.346661014776726 1.781064725250609 1.5965217213472793
- joint 14_to_0: origin xyz=0.9519997554499254 0.8346274683241105 0.9807371605957307 rpy=3.519991522165089 1.781064725250609 1.5965217213472793 -> xyz=0.9999 0.8346274683241105 0.9807371605957307 rpy=3.519991522165089 1.781064725250609 1.5965217213472793
- joint 22_to_11: origin xyz=0.09578858548659108 0.4421603294737 0.1263421961644826 rpy=0.6205493639575665 5.1512966192912 2.8832054081695433 -> xyz=0.1957885854865911 0.4421603294737 0.1263421961644826 rpy=0.6205493639575665 5.1512966192912 2.8832054081695433
- joint 23_to_11: origin xyz=0.09578858548659108 0.4421603294737 0.1263421961644826 rpy=0.9308240459363498 5.1512966192912 2.8832054081695433 -> xyz=0.1957885854865911 0.4421603294737 0.1263421961644826 rpy=0.9308240459363498 5.1512966192912 2.8832054081695433
- joint 25_to_14: origin xyz=0.09578858548659108 0.4421603294737 0.1263421961644826 rpy=0.6205493639575665 5.1512966192912 2.8832054081695433 -> xyz=0.1957885854865911 0.4421603294737 0.1263421961644826 rpy=0.6205493639575665 5.1512966192912 2.8832054081695433
- joint 26_to_14: origin xyz=0.09578858548659108 0.4421603294737 0.1263421961644826 rpy=0.9308240459363498 5.1512966192912 2.8832054081695433 -> xyz=0.1957885854865911 0.4421603294737 0.1263421961644826 rpy=0.9308240459363498 5.1512966192912 2.8832054081695433
